File: core.kicad_pcb (KiCad board)
At the start: 2 copper layers, 0 parts

Commit message: WIP
Parts:
- added AU1: AUDIO OUT, LIBS:Medved_Jack_3.5mm_CUI_SJ1-3535NG_Horizontal, F.Cu at (153.1, 49.8)
- added C1: 100n, LIBS:Medved_C_0805, F.Cu at (169.0, 79.8)
- added C10: 100n, LIBS:Medved_C_0805, F.Cu at (167.0, 79.8)
- added C11: 100n, LIBS:Medved_C_0805, F.Cu at (157.4, 74.6)
- added C12: 15p, LIBS:Medved_C_0805, F.Cu at (158.7, 79.7)
- added C13: 15p, LIBS:Medved_C_0805, F.Cu at (162.0, 82.6)
- added C14: 100n, LIBS:Medved_C_0805, F.Cu at (154.7, 65.8)
- added C15: 10u, LIBS:Medved_C_0805, F.Cu at (180.9, 60.4)
- added C16: 10u, LIBS:Medved_C_0805, F.Cu at (178.9, 60.3)
- added C17: 0.1u, LIBS:Medved_C_0805, F.Cu at (145.2, 64.0)
- added C18: 0.1u, LIBS:Medved_C_0805, F.Cu at (164.3, 59.8)
- added C19: 10u, LIBS:Medved_CP_Radial_D5.0mm_P2.50mm, F.Cu at (131.8, 74.2)
- added C2: 100n, LIBS:Medved_C_0805, F.Cu at (168.2, 59.8)
- added C20: 10u, LIBS:Medved_CP_Radial_D5.0mm_P2.50mm, F.Cu at (124.9, 74.2)
- added C21: 10n, LIBS:Medved_C_0805, F.Cu at (136.2, 69.5)
- added C22: 10n, LIBS:Medved_C_0805, F.Cu at (123.5, 69.5)
- added C23: 10u, LIBS:Medved_CP_Radial_D5.0mm_P2.50mm, F.Cu at (127.4, 82.9)
- added C24: 0.1u, LIBS:Medved_C_0805, F.Cu at (181.5, 82.6)
- added C25: 0.1u, LIBS:Medved_C_0805, B.Cu at (184.8, 73.0)
- added C3: 1u, LIBS:Medved_C_0805, F.Cu at (159.9, 64.2)
- added C4: 100n, LIBS:Medved_C_0805, F.Cu at (169.8, 64.2)
- added C5: 1u, LIBS:Medved_C_0805, F.Cu at (163.9, 64.2)
- added C6: 100n, LIBS:Medved_C_0805, F.Cu at (171.8, 64.2)
- added C7: 100n, LIBS:Medved_C_0805, F.Cu at (171.9, 69.5)
- added C8: 100n, LIBS:Medved_C_0805, F.Cu at (161.9, 64.2)
- added C9: 100n, LIBS:Medved_C_0805, F.Cu at (171.9, 73.5)
- added D1: 3V3, LIBS:Medved_D_0805, F.Cu at (154.2, 78.0)
- added D2: 3V3, LIBS:Medved_D_0805, F.Cu at (154.2, 80.2)
- added D3: 3V3, LIBS:Medved_D_0805, F.Cu at (154.2, 82.5)
- added D4: 3V3, LIBS:Medved_D_0805, F.Cu at (154.2, 84.8)
- added FL1: W25Q128JVS, LIBS:Medved_SOIC-8_5.23x5.23mm_P1.27mm, F.Cu at (153.2, 70.2)
- added H1: MountingHole, MountingHole:MountingHole_2.7mm, F.Cu at (124.8, 51.4)
- added H2: MountingHole, MountingHole:MountingHole_2.7mm, F.Cu at (189.4, 51.4)
- added H3: MountingHole, MountingHole:MountingHole_2.7mm, F.Cu at (189.4, 91.6)
- added H4: MountingHole, MountingHole:MountingHole_2.7mm, F.Cu at (124.8, 91.8)
- added HDMI1: HDMI, LIBS:HDMI, F.Cu at (184.2, 72.0)
- added JOY1: Joystick, LIBS:DSUB-9, F.Cu at (140.2, 87.3)
- added JOY2: Joystick, LIBS:DSUB-9, F.Cu at (174.4, 87.3)
- added JP1: Audio Jumpers, LIBS:Medved_JMP_2x03, F.Cu at (139.1, 72.8)
- added JP2: I2S, LIBS:Medved_PinHeader_1x02, F.Cu at (144.3, 72.8)
- added JP3: JMP PSRAM, Jumper:SolderJumper-2_P1.3mm_Open_RoundedPad1.0x1.5mm, B.Cu at (177.5, 76.5)
- added KB1: PS/2, LIBS:Connector_Mini-DIN_Female_6Pin_2rows, F.Cu at (136.8, 57.0)
- added L1: LED, LIBS:Medved_L_0805, F.Cu at (177.4, 79.1)
- added L2: GREEN, LIBS:Medved_L_0805, F.Cu at (185.4, 86.1)
- added PSR1: PSRAM, Package_SO:SO-8_5.3x6.2mm_P1.27mm, B.Cu at (177.4, 71.1)
- added R1: 27, LIBS:Medved_R_0805, F.Cu at (165.9, 64.2)
- added R10: 1k, LIBS:Medved_R_0805, F.Cu at (139.8, 66.0)
- added R11: 100R, LIBS:Medved_R_0805, F.Cu at (136.0, 64.0)
- added R12: 100R, LIBS:Medved_R_0805, F.Cu at (139.8, 64.0)
- added R13: 330R, LIBS:Medved_R_0805, F.Cu at (161.5, 57.5)
- added R14: 330R, LIBS:Medved_R_0805, F.Cu at (170.2, 57.5)
- added R15: 1k, LIBS:Medved_R_0805, F.Cu at (136.2, 78.5)
- added R16: 2k, LIBS:Medved_R_0805, F.Cu at (129.2, 69.5)
- added R17: 2k, LIBS:Medved_R_0805, F.Cu at (129.5, 78.8)
- added R18: 1k, LIBS:Medved_R_0805, F.Cu at (123.0, 78.8)
- added R19: 1k, LIBS:Medved_R_0805, F.Cu at (140.5, 83.2)
- added R2: 27, LIBS:Medved_R_0805, F.Cu at (167.8, 64.2)
- added R20: 1k, LIBS:Medved_R_0805, F.Cu at (174.8, 83.2)
- added R21: 270R, LIBS:Medved_R_0805, F.Cu at (177.4, 73.1)
- added R22: 270R, LIBS:Medved_R_0805, F.Cu at (177.4, 65.4)
- added R23: 270R, LIBS:Medved_R_0805, F.Cu at (177.4, 77.0)
- added R24: 270R, LIBS:Medved_R_0805, F.Cu at (177.4, 71.1)
- added R25: 270R, LIBS:Medved_R_0805, F.Cu at (177.4, 69.2)
- added R26: 270R, LIBS:Medved_R_0805, F.Cu at (177.4, 63.5)
- added R27: 270R, LIBS:Medved_R_0805, F.Cu at (177.4, 75.0)
- added R28: 270R, LIBS:Medved_R_0805, F.Cu at (177.4, 67.3)
- added R3: 1k, LIBS:Medved_R_0805, F.Cu at (150.7, 65.8)
- added R4: 1K, LIBS:Medved_R_0805, F.Cu at (171.0, 79.8)
- added R5: 1k, LIBS:Medved_R_0805, F.Cu at (165.0, 79.8)
- added R6: 5.1K, LIBS:Medved_R_0805, F.Cu at (176.9, 60.3)
- added R7: 5.1K, LIBS:Medved_R_0805, F.Cu at (174.9, 60.3)
- added R8: 1K, LIBS:Medved_R_0805, F.Cu at (185.3, 82.6)
- added R9: 1k, LIBS:Medved_R_0805, F.Cu at (136.0, 66.0)
- added RP1: RP2040, LIBS:RP2040-QFN-56, F.Cu at (164.9, 72.0)
- added SD1: 47571-0001, LIBS:microsd, F.Cu at (166.1, 51.8)
- added SW1: Flash Button, LIBS:Button_SMD_3x3x2, F.Cu at (122.7, 60.6)
- added SW2: Reset Button, LIBS:Button_SMD_3x3x2, F.Cu at (191.7, 82.5)
- added TDA1: TDA1387T, Package_SO:SO-8_5.3x6.2mm_P1.27mm, B.Cu at (154.5, 72.5)
- added U1: NCP1117-3.3_SOT223, LIBS:Medved_SOT-223-3_TabPin2, F.Cu at (187.3, 59.6)
- added USB1: USB Type C, LIBS:USB-TYPE-C-31-M-12_lib2, F.Cu at (178.8, 47.2)
- added Y1: ABM8-272-T3, Crystal:Crystal_SMD_3225-4Pin_3.2x2.5mm, F.Cu at (161.9, 79.8)
Routing:
- net VBUS: track 0.00 -> 190.6 mm, vias 0 -> 7
- net +3V3: track 0.00 -> 161.0 mm, vias 0 -> 1
- net Net-(RP1-VREG_VOUT): track 0.00 -> 6.40 mm
Other:
- board outline added: 70.6 x 46.2 mm

Commit message: Updates
Parts:
- C22, D1, D2, R10, R11, R12, R16, R17, R18, R9: moved to B.Cu
- moved SW2 65.2 mm to (126.8, 88.2), turned to 180 degrees
- moved C20 63.1 mm to (187.6, 67.4), turned to 90 degrees
- moved C24 59.6 mm to (126.6, 59.4)
- moved R18 59.5 mm to (181.6, 68.6), turned to 0 degrees
- moved C22 58.3 mm to (181.6, 64.6), turned to 180 degrees
- moved C19 55.6 mm to (187.4, 73.6), turned to 90 degrees
- moved HDMI1 54.7 mm to (129.6, 71.3), turned to -90 degrees
- moved R17 52.7 mm to (181.6, 70.6), turned to 180 degrees
- moved R16 52.4 mm to (181.6, 66.6), turned to 180 degrees
- moved JP1 51.7 mm to (189.4, 84.5), turned to 180 degrees
- moved C21 51.5 mm to (187.0, 60.8), turned to 180 degrees
- moved C23 50.4 mm to (177.1, 74.6), turned to 0 degrees
- moved R15 44.4 mm to (180.6, 80.0)
- moved R26 43.6 mm to (136.6, 78.9), turned to 0 degrees
- moved R22 42.4 mm to (136.6, 77.0), turned to 0 degrees
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Routing:
- net /GP_J3: track 0.00 -> 73.0 mm
- net /GP_J4: track 0.00 -> 61.1 mm, vias 0 -> 6
- net +3V3: track 161.0 -> 219.7 mm, vias 1 -> 12
- net Net-(KB1-Pad5): track 0.00 -> 56.7 mm, vias 0 -> 5
- net /RP2040/QSPI_SS: track 0.00 -> 50.7 mm
- net /RUN: track 0.00 -> 49.3 mm, vias 0 -> 8
- net /SD_DAT3: track 0.00 -> 49.1 mm, vias 0 -> 2
- net /AU_DATA: track 0.00 -> 42.8 mm, vias 0 -> 4
- net VBUS: track 190.6 -> 233.1 mm
- net /SD_DAT0: track 0.00 -> 38.6 mm, vias 0 -> 2
- net Net-(KB1-Pad1): track 0.00 -> 36.6 mm, vias 0 -> 1
- net /AU_SCLK: track 0.00 -> 35.6 mm, vias 0 -> 3
- net /SD_CMD: track 0.00 -> 34.1 mm, vias 0 -> 2
- net /SD_CLK: track 0.00 -> 31.7 mm, vias 0 -> 2
- net /AU_LRCK: track 0.00 -> 31.2 mm, vias 0 -> 1
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Other:
- outline, holes or cut-outs redrawn

Commit message: HW Rev 1.0
Parts:
- added C26: 100n, LIBS:Medved_C_0805, F.Cu at (168.4, 78.0)
- JP3: footprint Jumper:SolderJumper-2_P1.3mm_Open_RoundedPad1.0x1.5mm -> LIBS:Medved_Jumper_Solder
- Y1: value ABM8-272-T3 -> 12 MHz; footprint Crystal:Crystal_SMD_3225-4Pin_3.2x2.5mm -> LIBS:Medved_CRYSTAL_3225
- moved C18 46.7 mm to (126.6, 57.4), turned to 0 degrees
- moved JP1 5.72 mm to (186.9, 79.4), turned to 0 degrees
- moved JP2 5.13 mm to (184.2, 79.4), turned to 0 degrees
- moved R3 2.22 mm to (132.8, 82.1)
- moved SW2 0.81 mm to (126.8, 89.0)
Routing:
- net /AU_DATA: track 42.8 -> 55.7 mm
- net /Audio/RIGHT_OUT: track 23.9 -> 14.4 mm
- net /Audio/BEEP_OUT: track 21.2 -> 30.7 mm
- net +3V3: track 219.7 -> 227.6 mm
- net /AU_LRCK: track 31.2 -> 37.9 mm
- net /Audio/RIGHT_TDA: track 19.6 -> 24.9 mm
- net /RP2040/QSPI_SS: track 50.7 -> 53.7 mm
- net /RP2040/~{USB_BOOT}: track 6.15 -> 9.04 mm
- net /AU_SCLK: track 35.6 -> 34.5 mm
- net /Audio/LEFT_OUT: track 10.8 -> 11.5 mm, vias 0 -> 1
- net /GP_J4: track 61.1 -> 61.8 mm
- net VBUS: track 233.1 -> 232.4 mm
- net GND: vias 34 -> 39
Other:
- outline, holes or cut-outs redrawn
- board text added: "BEEP"
- board text added: "BOOT"
- board text added: "CORE"
- board text added: "HW REV 1.0"
- board text added: "L"
- board text added: "PWM"
- board text added: "R"
- board text added: "RESET"
- board text added: "RH1.DEV"
- board text added: "TDA"
