File: core.kicad_sch (KiCad schematic)
At the start: 0 parts

Commit message: WIP
Parts:
- added H1, H2, H3, H4: MountingHole, MountingHole:MountingHole_2.7mm, symbol Mechanical:MountingHole
Connections:
- no-connect marks 22 -> 10
Other:
- added sheet HDMI (hdmi.kicad_sch)
- added sheet PSRAM (psram.kicad_sch)
