File: gamepad.kicad_sch (KiCad schematic)
At the start: 3 parts

Commit message: WIP
Parts:
- JOY1: renamed from JOY2; footprint LIBS:DB9 -> LIBS:DSUB-9
- renumbered D4 to D3, R20 to R19
Changed lines of the file:
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@@
 		(on_board yes)
 		(dnp no)
-		(property "Reference" "#PWR047"
+		(property "Reference" "#PWR044"
 			(at 63.5 76.2 0)
 			(effects
@@
 		(on_board yes)
 		(dnp no)
-		(property "Reference" "D4"
+		(property "Reference" "D3"
 			(at 60.96 64.77 0)
 			(effects
@@
 		(dnp no)
 		(fields_autoplaced yes)
-		(property "Reference" "#PWR048"
+		(property "Reference" "#PWR045"
 			(at 76.2 58.42 0)
 			(effects
@@
 		(on_board yes)
 		(dnp no)
-		(property "Reference" "JOY2"
+		(property "Reference" "JOY1"
 			(at 93.98 41.91 0)
 			(effects
@@
 			)
 		)
-		(property "Footprint" "LIBS:DB9"
+		(property "Footprint" "LIBS:DSUB-9"
 			(at 92.71 54.61 0)
 			(effects
@@
 		(dnp no)
 		(fields_autoplaced yes)
-		(property "Reference" "#PWR049"
+		(property "Reference" "#PWR046"
 			(at 71.12 52.07 0)
 			(effects
@@
 		(on_board yes)
 		(dnp no)
-		(property "Reference" "R20"
+		(property "Reference" "R19"
 			(at 66.04 57.15 90)
 			(effects

Commit message: HW Rev 1.0
Other:
- title: FRANK -> CORE
Changed lines of the file:
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@@
 	(generator "eeschema")
 	(generator_version "8.0")
-	(paper "A4")
+	(paper "A3")
 	(title_block
-		(title "FRANK")
-		(date "2024-12-15")
-		(rev "2.0")
+		(title "CORE")
+		(date "2024-12-17")
+		(rev "1.0")
 		(company "Mikhail Matveev")
-		(comment 1 "https://github.com/xtremespb/frank2")
+		(comment 1 "https://github.com/xtremespb/core")
 	)
 	(junction
