File: hdmi.kicad_sch (KiCad schematic)
At the start: 10 parts

Commit message: HW Rev 1.0
Parts:
- renumbered C2 to C24, R5 to R21, R6 to R22, R7 to R23, R8 to R24, R9 to R25, R10 to R26, R11 to R27, R12 to R28
Other:
- title: FRANK -> CORE
Changed lines of the file:
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@@
 	(generator "eeschema")
 	(generator_version "8.0")
-	(paper "A4")
+	(paper "A3")
 	(title_block
-		(title "FRANK")
-		(date "2024-12-15")
-		(rev "2.0")
+		(title "CORE")
+		(date "2024-12-17")
+		(rev "1.0")
 		(company "Mikhail Matveev")
-		(comment 1 "https://github.com/xtremespb/frank2")
+		(comment 1 "https://github.com/xtremespb/core")
 	)
 	(junction
@@
 		(on_board yes)
 		(dnp no)
-		(property "Reference" "R8"
+		(property "Reference" "R24"
 			(at 87.63 91.44 90)
 			(effects
@@
 		(on_board yes)
 		(dnp no)
-		(property "Reference" "R12"
+		(property "Reference" "R28"
 			(at 97.79 99.06 90)
 			(effects
@@
 		(on_board yes)
 		(dnp no)
-		(property "Reference" "R7"
+		(property "Reference" "R23"
 			(at 87.63 78.74 90)
 			(effects
@@
 		(on_board yes)
 		(dnp no)
-		(property "Reference" "R9"
+		(property "Reference" "R25"
 			(at 87.63 93.98 90)
 			(effects
@@
 		(on_board yes)
 		(dnp no)
-		(property "Reference" "C2"
+		(property "Reference" "C24"
 			(at 73.7616 61.849 0)
 			(effects
@@
 		(on_board yes)
 		(dnp no)
-		(property "Reference" "R5"
+		(property "Reference" "R21"
 			(at 77.47 86.36 90)
 			(effects
@@
 		(dnp no)
 		(fields_autoplaced yes)
-		(property "Reference" "#PWR012"
+		(property "Reference" "#PWR051"
 			(at 64.77 124.46 0)
 			(effects
@@
 		(on_board yes)
 		(dnp no)
-		(property "Reference" "R11"
+		(property "Reference" "R27"
 			(at 97.79 83.82 90)
 			(effects
@@
 		(on_board yes)
 		(dnp no)
-		(property "Reference" "R10"
+		(property "Reference" "R26"
 			(at 87.63 106.68 90)
 			(effects
@@
 		(on_board yes)
 		(dnp no)
-		(property "Reference" "R6"
+		(property "Reference" "R22"
 			(at 77.47 101.6 90)
 			(effects
