File: reset.kicad_sch (KiCad schematic)
At the start: 1 part, among them SW1 Reset Button

Commit message: WIP
Parts:
- renumbered SW1 to SW2
Changed lines of the file:
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@@
 		(on_board yes)
 		(dnp no)
-		(property "Reference" "SW1"
+		(property "Reference" "SW2"
 			(at 62.484 49.022 0)
 			(effects
@@
 		(dnp no)
 		(fields_autoplaced yes)
-		(property "Reference" "#PWR029"
+		(property "Reference" "#PWR050"
 			(at 48.26 41.91 0)
 			(effects

Commit message: HW Rev 1.0
Other:
- title: FRANK2 -> CORE
Changed lines of the file:
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@@
 	(generator "eeschema")
 	(generator_version "8.0")
-	(paper "A4")
+	(paper "A3")
 	(title_block
-		(title "FRANK2")
-		(date "2024-11-21")
+		(title "CORE")
+		(date "2024-12-17")
 		(rev "1.0")
 		(company "Mikhail Matveev")
-		(comment 1 "https://github.com/xtremespb/frank2")
+		(comment 1 "https://github.com/xtremespb/core")
 	)
 	(junction
