File: rp2040.kicad_sch (KiCad schematic)
At the start: 24 parts, among them SW1 Flash Button, Y1 ABM8-272-T3

Commit message: HW Rev 1.0
Parts:
- added C26: 100n, LIBS:Medved_C_0805, symbol Device:C
- Y1: value ABM8-272-T3 -> 12 MHz; footprint Crystal:Crystal_SMD_3225-4Pin_3.2x2.5mm -> LIBS:Medved_CRYSTAL_3225
Connections:
- net +3V3: now also C26.1
- net GND: now also C26.2
Changed lines of the file:
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@@
 	(title_block
 		(title "CORE")
-		(date "2024-12-16")
+		(date "2024-12-17")
 		(rev "1.0")
 		(company "Mikhail Matveev")
-		(comment 1 "https://github.com/xtremespb/frank2")
+		(comment 1 "https://github.com/xtremespb/core")
 	)
 	(junction
@@
 	)
 	(junction
+		(at 170.18 38.1)
+		(diameter 0)
+		(color 0 0 0 0)
+	)
+	(junction
 		(at 82.55 58.42)
 		(diameter 0)
@@
 	(wire
 		(pts
+			(xy 181.61 39.37) (xy 181.61 38.1)
+		)
+		(stroke
+			(width 0)
+			(type default)
+		)
+	)
+	(wire
+		(pts
 			(xy 107.95 142.24) (xy 123.19 142.24)
 		)
@@
 	(wire
 		(pts
+			(xy 181.61 46.99) (xy 181.61 49.53)
+		)
+		(stroke
+			(width 0)
+			(type default)
+		)
+	)
+	(wire
+		(pts
 			(xy 201.93 68.58) (xy 203.2 68.58)
 		)
@@
 	(wire
 		(pts
+			(xy 170.18 38.1) (xy 181.61 38.1)
+		)
+		(stroke
+			(width 0)
+			(type default)
+		)
+	)
+	(wire
+		(pts
 			(xy 208.28 116.84) (xy 205.74 116.84)
 		)
@@
 	(wire
 		(pts
+			(xy 170.18 49.53) (xy 181.61 49.53)
+		)
+		(stroke
+			(width 0)
+			(type default)
+		)
+	)
+	(wire
+		(pts
 			(xy 55.88 58.42) (xy 55.88 71.12)
 		)
@@
 			)
 		)
-		(property "Value" "ABM8-272-T3"
+		(property "Value" "12 MHz"
 			(at 220.98 104.14 90)
 			(effects
@@
 			)
 		)
-		(property "Footprint" "Crystal:Crystal_SMD_3225-4Pin_3.2x2.5mm"
+		(property "Footprint" "LIBS:Medved_CRYSTAL_3225"
 			(at 227.33 111.76 0)
 			(effects
@@
 			)
 		)
-		(property "Description" ""
+		(property "Description" "ABM8-272-T3"
 			(at 227.33 111.76 0)
 			(effects
@@
 					(unit 1)
 				)
+			)
+		)
+	)
+	(symbol
+		(lib_id "Device:C")
+		(at 181.61 43.18 0)
+		(unit 1)
+		(exclude_from_sim no)
+		(in_bom yes)
+		(on_board yes)
+		(dnp no)
+		(property "Reference" "C26"
+			(at 184.531 42.0116 0)
+			(effects
+				(font
+					(size 1.27 1.27)
+				)
+				(justify left)
+			)
+		)
+		(property "Value" "100n"
+			(at 184.531 44.323 0)
+			(effects
+				(font
+					(size 1.27 1.27)
+				)
+				(justify left)
+			)
+		)
+		(property "Footprint" "LIBS:Medved_C_0805"
+			(at 182.5752 46.99 0)
+			(effects
+				(font
+					(size 1.27 1.27)
+				)
+				(hide yes)
+			)
+		)
+		(property "Datasheet" "~"
+			(at 181.61 43.18 0)
+			(effects
+				(font
+					(size 1.27 1.27)
+				)
+				(hide yes)
+			)
+		)
+		(property "Description" ""
+			(at 181.61 43.18 0)
+			(effects
+				(font
+					(size 1.27 1.27)
+				)
+				(hide yes)
+			)
+		)
+		(pin "1"
+		)
+		(pin "2"
+		)
+		(instances
+			(project "core"
+				(path "/8c0b3d8b-46d3-4173-ab1e-a61765f77d61/b0409f8e-084a-4c18-99f6-a5d70280ca34"
+					(reference "C26")
+					(unit 1)
+				)
